File: CellCTRL_MPC01/MPC-Servo/MPC_Servo/MPC_Servo.kicad_pcb (KiCad board)
At the start: 2 copper layers, 35 x 25 mm, 16 parts, among them J1 Programming, J2 I2C, J3 Reset, J4 Servo_1, J5 Servo_2/NC, J6 Power, U1 ATtiny202-SS

Commit message: Fertig V0.1_Servo
Parts:
- J2: footprint Connector_JST:JST_EH_B4B-EH-A_1x04_P2.50mm_Vertical -> Connector_JST:JST_XH_B4B-XH-A_1x04_P2.50mm_Vertical
- J4: footprint Connector_JST:JST_PH_B3B-PH-K_1x03_P2.00mm_Vertical -> Connector_JST:JST_XH_B3B-XH-A_1x03_P2.50mm_Vertical
- J5: value Servo_2/NC -> Servo_2/Endstop; footprint Connector_JST:JST_PH_B3B-PH-K_1x03_P2.00mm_Vertical -> Connector_JST:JST_XH_B3B-XH-A_1x03_P2.50mm_Vertical
- J6: value Power -> Power/Servo; footprint Connector_PinHeader_2.54mm:PinHeader_1x02_P2.54mm_Vertical -> Connector_JST:JST_XH_B2B-XH-A_1x02_P2.50mm_Vertical
- moved J5 4.61 mm to (126.0, 71.5), turned to 90 degrees
- moved H2 2.50 mm to (127.0, 49.5)
- moved H1 1.50 mm to (152.0, 71.5)
- moved J3 1.50 mm to (151.5, 58.0)
- moved J4 1.50 mm to (126.0, 60.5)
- moved J6 1.00 mm to (136.0, 51.0), turned to 180 degrees
- moved F1 0.80 mm to (132.4, 55.8)
Routing:
- net Net-(J5-Pin_1): track 9.66 -> 15.4 mm
- net Net-(J6-Pin_2): track 3.01 -> 4.83 mm
- net GND: track 15.9 -> 17.4 mm
- net Reset: track 9.37 -> 10.9 mm
- net VCC: track 23.2 -> 21.8 mm
- net Net-(J4-Pin_1): track 8.24 -> 7.62 mm
Other:
- board size 35 x 25 mm -> 35 x 30 mm
- board text added: "5V"
- board text added: "Controller Servo(CellCTRL) V0.1 03/2026 Edit by JK github.com/Kappi084/CellCTRL"
- board text added: "Data"
- board text added: "GND"
- board text added: "PRG"
- board text added: "RST"
- board text added: "SCL"
- board text added: "SDA"
- board text added: "VCC"
- board text added: "VCC-IN"
- board text removed: "Edit by JK V0.1"
